File: eagle/pinoccio-motion.sch (EAGLE design)
At the start: 3 parts

Commit message: updated motion to v0.1
Parts:
- added C1: 1.0uf, Pinoccio:CAP0402-CAP
- added C2, C6: 0.01uf, Pinoccio:CAP0402-CAP
- added C3: 2.2nf, Pinoccio:CAP0603-CAP
- added C4, C5, C7, C8: 0.1uf, Pinoccio:CAP0402-CAP
- added J1: AVR_SPI_PRG_6, Pinoccio:AVR_SPI_PRG_6
- added JP1, JP2, JP3: (no value), Pinoccio:JUMPER-2SMD-NC
- added R1, R2, R3: 100K, Pinoccio:RESISTOR0402-RES
- added R4, R5: 1K, Pinoccio:RESISTOR0402-RES
- added U$2: MS5611, Pinoccio:MS5611
- added U$3: SWITCH-MOSFETTDFN4, Pinoccio:SWITCH-MOSFETTDFN4
- added U$4: U.FL, Pinoccio:U.FL
- added U1: ATTINY13QFN10, Pinoccio:ATTINY13QFN10
- added U2: MPU-9150, Pinoccio:MPU-9150QFN-24-NP
- U$1: value PROTO -> FGPMMOPA6H; device Pinoccio:PROTO -> Pinoccio:FGPMMOPA6H
Connections:
- removed net D0: JP-L.10
- removed net D1: JP-L.11
- removed net VBAT-AE: JP-R.3, U$1.P-VBAT
- new net BKPK-BUS: J1.1, JP-L.2, U1.PB1(MISO)
- new net D7: JP-L.15, JP1.2
- new net D8: JP-L.16, JP3.1
- new net GPS-EN: R3.2, U$3.ON, U1.PB4(ADC2)
- new net N$1: J1.4, U1.PB0(MOSI)
- new net N$10: JP3.2, U$1.1PPS
- new net N$11: C4.1, U2.REGOUT
- new net N$2: R4.1, U$1.RX
- new net N$3: J1.3, U1.PB2(SCK/ADC1)
- new net N$4: J1.5, R1.1, U1.PB5(NRES)
- new net N$5: U$1.EXT-ANT, U$4.SIGNAL
- new net N$6: R5.1, U$1.TX
- new net N$7: JP1.1, U2.INT
- new net N$8: C3.1, U2.CPOUT
- new net N$9: JP2.1, U$1.3D-FIX
- new net VBAT: JP-R.3, U$1.VBACKUP
- new net VCC-GPS: C1.1, C2.1, U$1.VCC, U$3.OUT
- net D2: now also JP-L.10; no longer JP-L.12
- net D3: now also JP-L.11; no longer JP-L.13
- net D4: now also JP-L.12; no longer JP-L.14
- net D5: now also JP-L.13; no longer JP-L.15
- net D6: now also JP-L.14, JP2.2; no longer JP-L.16
- net GND: now also C1.2, C2.2, C3.2, C4.2, C5.2, C6.2, C7.2, C8.2, J1.6, R3.1, U$1.GND@12, U$1.GND@19, U$1.GND@3, U$1.GND@8, U$2.CSB, U$2.GND, U$3.GND, U$4.GND@0, U$4.GND@1, U1.GND, U2.AD0, U2.CLKIN, U2.FSYNC, U2.GND@15, U2.GND@17, U2.GND@18; no longer JP-L.2, U$1.P$53, U$1.P$77, U$1.P-GND, U$1.P-GND2
- net RESET: now also R2.1, U$1.~RESET; no longer U$1.P-RESET
- net RX1: now also R5.2
- net SCL: now also U$2.SCLK, U2.SCL
- net SDA: now also U$2.SDI/SDA, U2.SDA
- net TX1: now also R4.2
- net VCC-AE: now also C5.1, C6.1, C7.1, C8.1, J1.2, R1.2, R2.2, U$2.PS, U$2.VDD, U$3.IN, U1.VCC, U2.VDD@13, U2.VDD@3, U2.VLOGIC; no longer U$1.P-VCC
- net VUSB: no longer U$1.P-VUSB
Other:
- note added: "1.0"
- note removed: "0.9"
- moved on the sheet: JP-L, JP-R
