File: eagle/pinoccio-motion.sch (EAGLE design)
At the start: 25 parts, among them J1 AVR_SPI_PRG_6, U1 ATTINY13QFN10, U2 MPU-9150

Commit message: v0.2 fixes
Parts:
- removed C2: 0.01uf, Pinoccio:CAP0402-CAP
- removed U$3: SWITCH-MOSFETTDFN4, Pinoccio:SWITCH-MOSFETTDFN4
- added C9: 0.1uf, Pinoccio:CAP0402-CAP
- added LED1: (no value), Pinoccio:LED0603
- added R10, R9: 10k, Pinoccio:RESISTOR0402-RES
- added R6, R7, R8: 100k, Pinoccio:RESISTOR0402-RES
- added U3: M25PX16, Pinoccio:M25PX16SO8N
- C1: value 1.0uf -> 0.1uf
- R3: value 100K -> 1k
Connections:
- removed net GPS-EN: R3.2, U$3.ON, U1.PB4(ADC2)
- removed net VCC-GPS: C1.1, C2.1, U$1.VCC, U$3.OUT
- new net N$12: R7.2, U3.!WP
- new net N$13: R8.2, U3.!HOLD
- new net N$14: LED1.A, R3.1
- net D5: now also JP3.1
- net D8: no longer JP3.1
- net GND: now also C1.1, C9.2, LED1.C, U3.GND; no longer C1.2, C2.2, R3.1, U$3.GND
- net MISO: now also U3.SO
- net MOSI: now also U3.SI
- net N$9: now also R3.2
- net SCK: now also U3.SCK
- net SCL: now also R10.2
- net SDA: now also R9.2
- net SSN: now also R6.2, U3.!CS
- net VCC-AE: now also C1.2, C9.1, R10.1, R6.1, R7.1, R8.1, R9.1, U$1.VCC, U3.VCC; no longer U$3.IN
Other:
- note added: "0.3"
- note added: "Copyright Pinoccio 2012-2014"
- note removed: "1.0"
- note removed: "Copyright Pinoccio 2012-2013"
- moved on the sheet: C1, C7, C8, J1, JP2, R1, R2, R3, U$2, U1
