File: eagle/pinoccio-motion.brd (EAGLE design)
At the start: 25.4 x 42.7 mm, 25 parts, among them J1 AVR_SPI_PRG_6, U1 ATTINY13QFN10, U2 MPU-9150

Commit message: v0.2 fixes
Parts:
- removed C2: 0.01uf, Pinoccio:0402-CAP
- removed U$3: SWITCH-MOSFETTDFN4, Pinoccio:TDFN4
- added C9: 0.1uf, Pinoccio:0402-CAP
- added LED1: (no value), Pinoccio:LED-0603
- added R10, R9: 10k, Pinoccio:0402-RES
- added R6, R7, R8: 100k, Pinoccio:0402-RES
- added U3: M25PX16, Pinoccio:SO8N
- C1: value 1.0uf -> 0.1uf
- R3: value 100K -> 1k
- moved R4 15.8 mm to (15.3, 45.1), turned to 270 degrees
- moved R5 13.5 mm to (16.6, 45.1), turned to 270 degrees
- moved C1 12.9 mm to (1.80, 61.7), turned to 0 degrees
- moved U$1 12.5 mm to (4.80, 46.9)
- moved U$4 11.4 mm to (20.8, 43.0)
- moved R3 11.3 mm to (1.80, 56.2), turned to 270 degrees
- moved C7 8.88 mm to (10.2, 37.1)
- moved R1 8.57 mm to (15.2, 39.9), turned to 90 degrees
- moved U1 8.00 mm to (12.7, 38.6), turned to 180 degrees
- moved R2 6.24 mm to (8.51, 36.7)
- moved JP3 5.92 mm to (6.05, 15.4)
- moved C3 1.64 mm to (16.4, 23.6)
- moved U2 1.45 mm to (12.7, 21.4)
- moved C8 1.45 mm to (9.63, 15.0)
- moved U$2 1.45 mm to (11.2, 10.6)
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Connections:
- removed net GPS-EN: R3.2, U$3.P$4, U1.4
- removed net VCC-GPS: C1.1, C2.1, U$1.P$1, U$3.P$1
- new net N$12: R7.2, U3.3
- new net N$13: R8.2, U3.7
- new net N$14: LED1.A, R3.1
- net D5: now also JP3.1
- net D8: no longer JP3.1
- net GND: now also C1.1, C9.2, LED1.C, U3.4; no longer C1.2, C2.2, R3.1, U$3.P$2, U$3.P$5
- net MISO: now also U3.2
- net MOSI: now also U3.5
- net N$9: now also R3.2
- net SCK: now also U3.6
- net SCL: now also R10.2
- net SDA: now also R9.2
- net SSN: now also R6.2, U3.1
- net VCC-AE: now also C1.2, C9.1, R10.1, R6.1, R7.1, R8.1, R9.1, U$1.P$1, U3.8; no longer U$3.P$3
Routing:
- net SSN: track 0.00 -> 25.2 mm
- net N$9: track 33.4 -> 58.0 mm
- net VCC-AE: track 70.0 -> 90.6 mm
- net MOSI: track 0.00 -> 17.9 mm
- net SCK: track 0.00 -> 16.7 mm, vias 0 -> 2
- net GPS-EN: track 16.6 -> 0.00 mm
- net MISO: track 0.00 -> 16.2 mm
- net TX1: track 2.45 -> 16.7 mm
- net VBAT: track 27.1 -> 41.3 mm, vias 1 -> 2
- net N$3: track 17.7 -> 4.02 mm
- net BKPK-BUS: track 25.1 -> 12.0 mm, vias 0 -> 1
- net RESET: track 22.6 -> 35.3 mm, vias 2 -> 4
- net RX1: track 2.45 -> 14.2 mm
- net N$2: track 21.3 -> 13.6 mm, vias 2 -> 0
- net N$4: track 11.3 -> 3.86 mm
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Other:
- board size 25.4 x 42.7 mm -> 25.4 x 55.4 mm
- board text added: "2014-09-19"
- board text added: "Pinoccio(tm) Motion Backpack v0.3"
- board text added: "motion backpack v0.3"
- board text removed: "2013-09-26"
- board text removed: "Pinoccio(tm) Motion Backpack v0.1"
- board text removed: "motion backpack v0.1"
